Commit message: Correct some offsets

File: turtlebot_description/robots/turtlebot_radio_xtion_hokuyo.urdf.xacro (robot description, xacro)
@@ -22,6 +22,6 @@
   <!--sensor_asus_xtion_pro   		  parent="telescopic_camera_frame"/-->
   <!--sensor_asus_xtion_pro_offset	  		  parent="telescopic_bar_link"/-->
-  <sensor_asus_xtion_pro_live  name="tb" parent="telescopic_link" >
-	<origin xyz="0 0 ${(pos_offset+foot_height)/2}" rpy="0 0 0" />
+  <sensor_asus_xtion_pro_live  name="tb" parent="telescopic_camera_link" >
+	<origin xyz="0 0.021 0" rpy="0 0 0" />
    </sensor_asus_xtion_pro_live>
    <sensor_hokuyo_urg04lx name="tb" parent="base_link" >

File: turtlebot_description/urdf/stacks/telescopic.urdf.xacro (robot description, xacro)
@@ -60,4 +60,10 @@
       </collision>
     </link>
+     <joint name="telescopic_camera_joint" type="fixed">
+      <origin xyz="0.0 0.0 0.03" rpy="0 0 0" />
+      <parent link="telescopic_foot_link"/>
+      <child link="telescopic_camera_link" />
+    </joint>
+    <link name="telescopic_camera_link"/>
   </xacro:macro>
   <xacro:macro name="stack_bar" params="parent">

Commit message: var changed

File: turtlebot_description/robots/turtlebot_radio_xtion_hokuyo.urdf.xacro (robot description, xacro)
@@ -7,12 +7,12 @@
 -->
 <robot name="turtlebot" xmlns:xacro="http://ros.org/wiki/xacro">
-  <xacro:property name="pos_offset" value="0.661" />
-  <xacro:property name="foot_height" value="0.015" />
+  <xacro:property name="camera_h" value="0.406" />
+  <xacro:property name="foot_h" value="0.015" />
   <!--
     - Defautl measured positions of telescopic bar (change at you own convenience)
-          pos 1: 0.411
-          pos 2: 0.661
-          pos 3: 0.926
-          pos 4: 1.211
+          pos 0: 0.406
+          pos 2: 0.671
+          pos 3: 0.961
+          pos 4: 1.236
 -->
   <xacro:include filename="$(find turtlebot_description)/urdf/turtlebot_library.urdf.xacro" />

File: turtlebot_description/urdf/stacks/telescopic.urdf.xacro (robot description, xacro)
@@ -50,5 +50,5 @@
         <origin xyz=" 0 0 0.007" rpy="0 0 0" />
         <geometry>
-           <cylinder length="${foot_height}" radius="0.015"/>
+           <cylinder length="${foot_h}" radius="0.015"/>
         </geometry>
       </visual>
@@ -56,5 +56,5 @@
         <origin xyz="0.0 0.0 0.007" rpy="0 0 0" />
         <geometry>
-          <cylinder length="${foot_height}" radius="0.015"/>
+          <cylinder length="${foot_h}" radius="0.015"/>
         </geometry>
       </collision>
@@ -68,5 +68,5 @@
   </xacro:macro>
   <xacro:macro name="stack_bar" params="parent">
-    <stack_telescopic_bar parent="${parent}" h_offset="${pos_offset}" x_loc= "-0.1" y_loc= "0.0" z_loc="0.19" />
+    <stack_telescopic_bar parent="${parent}" h_offset="${camera_h}" x_loc= "-0.1" y_loc= "0.0" z_loc="0.19" />
   </xacro:macro>
 </robot>

Commit message: fixed some scale issues

File: turtlebot_description/robots/turtlebot_radio_xtion_hokuyo.urdf.xacro (robot description, xacro)
@@ -24,5 +24,5 @@
   <sensor_asus_xtion_pro_live  name="tb" parent="telescopic_camera_link" >
 	<origin xyz="0 0.021 0" rpy="0 0 0" />
-   </sensor_asus_xtion_pro_live>
+  </sensor_asus_xtion_pro_live>
    <sensor_hokuyo_urg04lx name="tb" parent="base_link" >
 		<origin xyz="0.137 0 0.241" rpy="0 0 0" />

File: turtlebot_description/urdf/sensors/asus_xtion_pro_live.urdf.xacro (robot description, xacro)
@@ -2,8 +2,8 @@
 <robot name="sensor_asus_xtion_pro_live" xmlns:xacro="http://ros.org/wiki/xacro">
   <!-- Xacro properties -->
-  <xacro:property name="M_SCALE" value="0.001"/>
-  <xacro:property name="asus_xtion_pro_depth_rel_rgb_py" value="0.0270" />
-  <xacro:property name="asus_xtion_pro_cam_rel_rgb_py"   value="-0.0220" />
-  <xacro:property name="M_PI" value="3.1415926535897931" />
+  <property name="M_SCALE" value="0.001"/>
+  <property name="asus_xtion_pro_depth_rel_rgb_py" value="0.0270" />
+  <property name="asus_xtion_pro_cam_rel_rgb_py"   value="-0.0220" />
+  <property name="M_PI" value="3.1415926535897931" />
   <xacro:macro name="sensor_asus_xtion_pro_live" params="name parent *origin">
     <joint name="${name}_cam_rgb_joint" type="fixed">
@@ -45,6 +45,6 @@
         <origin xyz="-0.01 0 0" rpy="${-M_PI/2} -${M_PI} ${-M_PI/2}"/>
         <geometry>
-          <mesh filename="package://turtlebot_description/meshes/sensors/asus_xtion_pro_live.dae" scale="${M_SCALE} ${M_SCALE} ${M_SCALE}"/>
-        </geometry>
+          <mesh filename="package://turtlebot_description/meshes/sensors/xtion_camera.dae" scale="${M_SCALE} ${M_SCALE} ${M_SCALE}"/>
+        </geometry>_C
       </visual>
       <collision>

File: turtlebot_description/urdf/sensors/orbbec_astra.urdf.xacro (robot description, xacro)
@@ -1,6 +1,4 @@
 <?xml version="1.0"?>
 <robot name="sensor_orbbec_astra" xmlns:xacro="http://ros.org/wiki/xacro">
-  <!-- Xacro properties -->
-  <xacro:property name="M_SCALE" value="1.0"/>
   <!-- RGB sensor - cam -->
   <xacro:property name="orbbec_astra_cam_rel_rgb_px"   value="0.0" />

File: turtlebot_description/urdf/turtlebot_library.urdf.xacro (robot description, xacro)
@@ -14,7 +14,7 @@
   <xacro:include filename="$(find turtlebot_description)/urdf/stacks/hexagons.urdf.xacro"/>  <!-- dishes -->
   <!-- 3D Sensors -->
-  <xacro:include filename="$(find turtlebot_description)/urdf/sensors/kinect.urdf.xacro"/>
-  <xacro:include filename="$(find turtlebot_description)/urdf/sensors/asus_xtion_pro.urdf.xacro"/>
-  <xacro:include filename="$(find turtlebot_description)/urdf/sensors/asus_xtion_pro_offset.urdf.xacro"/>
+  <!--xacro:include filename="$(find turtlebot_description)/urdf/sensors/kinect.urdf.xacro"/-->
+  <!--xacro:include filename="$(find turtlebot_description)/urdf/sensors/asus_xtion_pro.urdf.xacro"/-->
+  <!--xacro:include filename="$(find turtlebot_description)/urdf/sensors/asus_xtion_pro_offset.urdf.xacro"/-->
   <xacro:include filename="$(find turtlebot_description)/urdf/sensors/asus_xtion_pro_live.urdf.xacro"/>
   <xacro:include filename="$(find turtlebot_description)/urdf/sensors/hokuyo_urg04lx.urdf.xacro" />
