Commit message: ADD model for tb and orbbec camera

File: turtlebot_description/robots/turtlebot_radio_orbbec_hokuyo.urdf.xacro (robot description, xacro)
@@ -22,8 +22,11 @@
   <!--sensor_asus_xtion_pro   		  parent="telescopic_camera_frame"/-->
   <!--sensor_asus_xtion_pro_offset	  		  parent="telescopic_bar_link"/-->
-  <sensor_asus_xtion_pro_live  name="tb" parent="telescopic_camera_link" >
+  <!--sensor_asus_xtion_pro_live  name="tb" parent="telescopic_camera_link" >
 	<origin xyz="0 0.021 0" rpy="0 0 0" />
-   </sensor_asus_xtion_pro_live>
-   <sensor_hokuyo_urg04lx name="tb" parent="base_link" >
+   </sensor_asus_xtion_pro_live-->
+   <sensor_orbbec_astra name="radio" parent="telescopic_camera_link">
+      <origin xyz="0 0.011 0" rpy="0 0 0" />
+   </sensor_orbbec_astra>
+   <sensor_hokuyo_urg04lx name="radio" parent="base_link" >
 		<origin xyz="0.137 0 0.241" rpy="0 0 0" />
    </sensor_hokuyo_urg04lx>

File: turtlebot_description/urdf/turtlebot_library.urdf.xacro (robot description, xacro)
@@ -19,4 +19,5 @@
   <xacro:include filename="$(find turtlebot_description)/urdf/sensors/asus_xtion_pro_live.urdf.xacro"/>
   <xacro:include filename="$(find turtlebot_description)/urdf/sensors/hokuyo_urg04lx.urdf.xacro" />
+  <xacro:include filename="$(find turtlebot_description)/urdf/sensors/orbbec_astra.urdf.xacro"/>
   <!-- Telescopic Bar -->
   <xacro:include filename="$(find turtlebot_description)/urdf/stacks/telescopic.urdf.xacro"/>

Commit message: fixed distances and offsets, colors

File: turtlebot_description/robots/turtlebot_radio_orbbec_hokuyo.urdf.xacro (robot description, xacro)
@@ -1,18 +1,22 @@
-<?xml version="1.0"?><!--
+<?xml version="1.0"?>
+<!--
     - Base      : kobuki
     - Stacks    : hexagons
     - Telescopic: telescopic
-    - 3d Sensor : xtion
+    - 3d Sensor : orbbec
     - Laser		: hokuyo
 -->
 <robot name="turtlebot" xmlns:xacro="http://ros.org/wiki/xacro">
-  <xacro:property name="camera_h" value="0.406" />
-  <xacro:property name="foot_h" value="0.015" />
-  <!--
-    - Defautl measured positions of telescopic bar (change at you own convenience)
-          pos 0: 0.406
-          pos 2: 0.671
-          pos 3: 0.961
-          pos 4: 1.236
+  <xacro:property name="CAMERA_H" value="0.197" />
+  <xacro:property name="FOOT_H" value="0.02" />
+<!--
+	- Distance from floot (base_footprint) to top_plate = 0.41 (41 cm)
+	- Distance from base_link to top_plate = 0.3996 (39.96 cm)
+	- Distance from middle plate to top plate = 0.2092 m (20.92 cm)
+    - Distance from top_plate to telescopic_bar foot:
+          pos 1: 0.197 m (19.7 cm)
+          pos 2: 0.457 m (45.7 cm)
+          pos 3: 0.725 m (72.5 cm)
+          pos 4: 0.974 m (97.4 cm)
 -->
   <xacro:include filename="$(find turtlebot_description)/urdf/turtlebot_library.urdf.xacro" />
@@ -20,16 +24,9 @@
   <stack_hexagons                 parent="base_link"/>
   <stack_bar				  	  parent="base_link"/>
-  <!--sensor_asus_xtion_pro   		  parent="telescopic_camera_frame"/-->
-  <!--sensor_asus_xtion_pro_offset	  		  parent="telescopic_bar_link"/-->
-  <!--sensor_asus_xtion_pro_live  name="tb" parent="telescopic_camera_link" >
-	<origin xyz="0 0.021 0" rpy="0 0 0" />
-   </sensor_asus_xtion_pro_live-->
-   <sensor_orbbec_astra name="radio" parent="telescopic_camera_link">
-      <origin xyz="0 0.011 0" rpy="0 0 0" />
-   </sensor_orbbec_astra>
-   <sensor_hokuyo_urg04lx name="radio" parent="base_link" >
+  <sensor_orbbec_astra name="radio" parent="telescopic_foot_link">
+      <origin xyz="0.02 0.011 ${2*FOOT_H-0.006}" rpy="0 0 0" />
+  </sensor_orbbec_astra>
+  <sensor_hokuyo_urg04lx name="radio" parent="base_link" >
 		<origin xyz="0.137 0 0.241" rpy="0 0 0" />
-   </sensor_hokuyo_urg04lx>
-  <!--sensor_asus_xtion_pro_offset   parent="base_link"/-->
-  <!--sensor_hokuyo   				  parent="base_link"/-->
+  </sensor_hokuyo_urg04lx>
 </robot>

File: turtlebot_description/robots/turtlebot_radio_xtion_hokuyo.urdf.xacro (robot description, xacro)
@@ -1,3 +1,4 @@
-<?xml version="1.0"?><!--
+<?xml version="1.0"?>
+<!--
     - Base      : kobuki
     - Stacks    : hexagons
@@ -7,12 +8,15 @@
 -->
 <robot name="turtlebot" xmlns:xacro="http://ros.org/wiki/xacro">
-  <xacro:property name="camera_h" value="0.406" />
-  <xacro:property name="foot_h" value="0.015" />
-  <!--
-    - Defautl measured positions of telescopic bar (change at you own convenience)
-          pos 0: 0.406
-          pos 2: 0.671
-          pos 3: 0.961
-          pos 4: 1.236
+  <xacro:property name="CAMERA_H" value="0.197" />
+  <xacro:property name="FOOT_H" value="0.02" />
+<!--
+	- Distance from floot (base_footprint) to top_plate = 0.41 (41 cm)
+	- Distance from base_link to top_plate = 0.3996 (39.96 cm)
+	- Distance from middle plate to top plate = 0.2092 m (20.92 cm)
+    - Distance from top_plate to telescopic_bar foot:
+          pos 1: 0.197 m (19.7 cm)
+          pos 2: 0.457 m (45.7 cm)
+          pos 3: 0.725 m (72.5 cm)
+          pos 4: 0.974 m (97.4 cm)
 -->
   <xacro:include filename="$(find turtlebot_description)/urdf/turtlebot_library.urdf.xacro" />
@@ -20,13 +24,9 @@
   <stack_hexagons                 parent="base_link"/>
   <stack_bar				  	  parent="base_link"/>
-  <!--sensor_asus_xtion_pro   		  parent="telescopic_camera_frame"/-->
-  <!--sensor_asus_xtion_pro_offset	  		  parent="telescopic_bar_link"/-->
-  <sensor_asus_xtion_pro_live  name="tb" parent="telescopic_camera_link" >
-	<origin xyz="0 0.021 0" rpy="0 0 0" />
+  <sensor_asus_xtion_pro_live  name="radio" parent="telescopic_foot_link" >
+	<origin xyz="0.018 0.021 ${2*FOOT_H-0.006}" rpy="0 0 0" />
   </sensor_asus_xtion_pro_live>
-   <sensor_hokuyo_urg04lx name="tb" parent="base_link" >
+  <sensor_hokuyo_urg04lx name="radio" parent="base_link" >
 		<origin xyz="0.137 0 0.241" rpy="0 0 0" />
-   </sensor_hokuyo_urg04lx>
-  <!--sensor_asus_xtion_pro_offset   parent="base_link"/-->
-  <!--sensor_hokuyo   				  parent="base_link"/-->
+  </sensor_hokuyo_urg04lx>
 </robot>

File: turtlebot_description/urdf/sensors/orbbec_astra.urdf.xacro (robot description, xacro)
@@ -49,5 +49,5 @@
         <origin xyz="0 0 0" rpy="0 0 0"/>
         <geometry>
-          <mesh filename="package://turtlebot_description/meshes/sensors/orbbec_astra.dae" scale="${M_SCALE} ${M_SCALE} ${M_SCALE}"/>
+          <mesh filename="package://turtlebot_description/meshes/sensors/orbbec_astra.dae" />
         </geometry>
       </visual>

File: turtlebot_description/urdf/stacks/telescopic.urdf.xacro (robot description, xacro)
@@ -1,4 +1,5 @@
 <?xml version="1.0"?>
 <robot name="telescopic_bar" xmlns:xacro="http://ros.org/wiki/xacro">
+  <xacro:property name="D_MID_TOP" value="0.2092" />
   <xacro:macro name="stack_telescopic_bar" params="parent h_offset x_loc y_loc z_loc">
     <joint name="telescopic_base_joint" type="fixed">
@@ -9,5 +10,5 @@
     <link name="telescopic_base_link"/>
     <joint name="telescopic_joint" type="fixed">
-      <origin xyz="0.0 0.0 ${h_offset/2}" rpy="0 0 0" />
+      <origin xyz="0.0 0.0 0.0" rpy="0 0 0" />
       <parent link="telescopic_base_link"/>
       <child link="telescopic_link" />
@@ -22,18 +23,19 @@
       </inertial>
       <visual>
-        <origin xyz=" 0 0 0.0" rpy="0 0 0" />
+        <origin xyz="0 0 ${((D_MID_TOP+h_offset)/2)-D_MID_TOP}" rpy="0 0 0" />
         <geometry>
-           <cylinder length="${h_offset}" radius="0.01"/>
+           <cylinder length="${D_MID_TOP+h_offset}" radius="0.01"/>
         </geometry>
+        <material name="material_black" />
       </visual>
       <collision>
-        <origin xyz="0.0 0.0 0.0" rpy="0 0 0" />
+        <origin xyz="0.0 0.0 0" rpy="0 0 0" />
         <geometry>
-          <cylinder length="${h_offset}" radius="0.01"/>
+          <cylinder length="${D_MID_TOP+h_offset}" radius="0.01"/>
         </geometry>
       </collision>
     </link>
     <joint name="telescopic_foot_joint" type="fixed">
-      <origin xyz="0.0 0.0 ${h_offset/2}" rpy="0 0 0" />
+      <origin xyz="0.0 0.0 ${h_offset}" rpy="0 0 0" />
       <parent link="telescopic_link"/>
       <child link="telescopic_foot_link" />
@@ -48,25 +50,20 @@
       </inertial>
       <visual>
-        <origin xyz=" 0 0 0.007" rpy="0 0 0" />
+        <origin xyz="0 0 ${FOOT_H/2}" rpy="0 0 0" />
         <geometry>
-           <cylinder length="${foot_h}" radius="0.015"/>
+           <cylinder length="${FOOT_H}" radius="0.015"/>
         </geometry>
+        <material name="material_black" />
       </visual>
       <collision>
-        <origin xyz="0.0 0.0 0.007" rpy="0 0 0" />
+        <origin xyz="0.0 0.0 ${FOOT_H/2}" rpy="0 0 0" />
         <geometry>
-          <cylinder length="${foot_h}" radius="0.015"/>
+          <cylinder length="${FOOT_H}" radius="0.015"/>
         </geometry>
       </collision>
     </link>
-     <joint name="telescopic_camera_joint" type="fixed">
-      <origin xyz="0.0 0.0 0.03" rpy="0 0 0" />
-      <parent link="telescopic_foot_link"/>
-      <child link="telescopic_camera_link" />
-    </joint>
-    <link name="telescopic_camera_link"/>
   </xacro:macro>
   <xacro:macro name="stack_bar" params="parent">
-    <stack_telescopic_bar parent="${parent}" h_offset="${camera_h}" x_loc= "-0.1" y_loc= "0.0" z_loc="0.19" />
+    <stack_telescopic_bar parent="${parent}" h_offset="${CAMERA_H}" x_loc= "-0.1" y_loc= "0.0" z_loc="0.3996" />
   </xacro:macro>
 </robot>

Commit message: description: adding microphone array and some adjustments

File: turtlebot_description/robots/turtlebot_radio_orbbec_hokuyo.urdf.xacro (robot description, xacro)
@@ -11,5 +11,5 @@
   <!--
     - Defautl measured positions of telescopic bar (change at you own convenience)
-          pos 0: 0.406
+          pos 1: 0.406
           pos 2: 0.671
           pos 3: 0.961
@@ -20,16 +20,15 @@
   <stack_hexagons                 parent="base_link"/>
   <stack_bar				  	  parent="base_link"/>
-  <!--sensor_asus_xtion_pro   		  parent="telescopic_camera_frame"/-->
-  <!--sensor_asus_xtion_pro_offset	  		  parent="telescopic_bar_link"/-->
-  <!--sensor_asus_xtion_pro_live  name="tb" parent="telescopic_camera_link" >
-	<origin xyz="0 0.021 0" rpy="0 0 0" />
-   </sensor_asus_xtion_pro_live-->
    <sensor_orbbec_astra name="radio" parent="telescopic_camera_link">
-      <origin xyz="0 0.011 0" rpy="0 0 0" />
+      <origin xyz="0.02 0.011 0" rpy="0 0 0" />
    </sensor_orbbec_astra>
    <sensor_hokuyo_urg04lx name="radio" parent="base_link" >
 		<origin xyz="0.137 0 0.241" rpy="0 0 0" />
    </sensor_hokuyo_urg04lx>
-  <!--sensor_asus_xtion_pro_offset   parent="base_link"/-->
-  <!--sensor_hokuyo   				  parent="base_link"/-->
+   <sensor_microphone_array name="radio" parent="plate_top_link" >
+		<origin xyz="0.08 0 0.005" rpy="0 0 0" />
+   </sensor_microphone_array>
+   <screen name="radio" parent="plate_top_link" >
+		<origin xyz="-0.03 0 0.05" rpy="0 -0.09 0" />
+   </screen>
 </robot>

File: turtlebot_description/robots/turtlebot_radio_xtion_hokuyo.urdf.xacro (robot description, xacro)
@@ -20,6 +20,4 @@
   <stack_hexagons                 parent="base_link"/>
   <stack_bar				  	  parent="base_link"/>
-  <!--sensor_asus_xtion_pro   		  parent="telescopic_camera_frame"/-->
-  <!--sensor_asus_xtion_pro_offset	  		  parent="telescopic_bar_link"/-->
   <sensor_asus_xtion_pro_live  name="tb" parent="telescopic_camera_link" >
 	<origin xyz="0 0.021 0" rpy="0 0 0" />
@@ -28,5 +26,6 @@
 		<origin xyz="0.137 0 0.241" rpy="0 0 0" />
    </sensor_hokuyo_urg04lx>
-  <!--sensor_asus_xtion_pro_offset   parent="base_link"/-->
-  <!--sensor_hokuyo   				  parent="base_link"/-->
+   <sensor_microphone_array name="radio" parent="plate_top_link" >
+		<origin xyz="0.08 0 0.005" rpy="0 0 0" />
+   </sensor_microphone_array>
 </robot>

File: turtlebot_description/urdf/sensors/orbbec_astra.urdf.xacro (robot description, xacro)
@@ -97,5 +97,5 @@
     </link>
   <!-- RGBD sensor for simulation, same as Kinect -->
-  <sensor_xtion_pro_gazebo/>
+  <sensor_orbbec_astra_gazebo/>
   </xacro:macro>
    <xacro:macro name="sensor_orbbec_astra_gazebo">

File: turtlebot_description/urdf/stacks/telescopic.urdf.xacro (robot description, xacro)
@@ -26,4 +26,7 @@
            <cylinder length="${h_offset}" radius="0.01"/>
         </geometry>
+        <material name="black">
+            <color rgba="0 0 0 1"/>
+        </material>
       </visual>
       <collision>
@@ -52,4 +55,7 @@
            <cylinder length="${foot_h}" radius="0.015"/>
         </geometry>
+         <material name="black">
+            <color rgba="0 0 0 1"/>
+        </material>
       </visual>
       <collision>

File: turtlebot_description/urdf/turtlebot_library.urdf.xacro (robot description, xacro)
@@ -22,3 +22,7 @@
   <!-- Telescopic Bar -->
   <xacro:include filename="$(find turtlebot_description)/urdf/stacks/telescopic.urdf.xacro"/>
+  <!-- Microphone Array -->
+  <xacro:include filename="$(find turtlebot_description)/urdf/sensors/microphone_array.urdf.xacro"/>
+  <!-- Others -->
+  <xacro:include filename="$(find turtlebot_description)/urdf/others/screen.urdf.xacro"/>
 </robot>

Commit message: Added rear cam model

File: turtlebot_description/robots/turtlebot_radio_orbbec_hokuyo.urdf.xacro (robot description, xacro)
@@ -27,4 +27,7 @@
       <origin xyz="0.02 0.011 ${2*FOOT_H-0.006}" rpy="0 0 0" />
   </sensor_orbbec_astra>
+  <sensor_logitech_c920 prefix="rear" parent="telescopic_foot_link">
+      <origin xyz="-0.02 0.011 0.049" rpy="0 0 0" />
+  </sensor_logitech_c920>
   <sensor_hokuyo_urg04lx name="hokuyo" parent="base_link" >
 		<origin xyz="0.137 0 0.241" rpy="0 0 0" />

File: turtlebot_description/urdf/turtlebot_library.urdf.xacro (robot description, xacro)
@@ -26,3 +26,4 @@
   <!-- Others -->
   <xacro:include filename="$(find turtlebot_description)/urdf/others/screen.urdf.xacro"/>
+  <xacro:include filename="$(find turtlebot_description)/urdf/sensors/logitech_c920.urdf.xacro"/>
 </robot>

Commit message: Changed distances

File: turtlebot_description/robots/turtlebot_radio_orbbec_hokuyo.urdf.xacro (robot description, xacro)
@@ -34,5 +34,5 @@
    </sensor_hokuyo_urg04lx>
    <sensor_microphone_array name="radio" parent="plate_top_link" >
-		<origin xyz="0.08 0 0.005" rpy="0 0 0" />
+		<origin xyz="0.1 0 0.006" rpy="0 0 0" />
    </sensor_microphone_array>
    <!--screen name="radio" parent="plate_top_link" >
