Commit message: description: adding min/max angle param for the ust10lx version

File: turtlebot_description/robots/turtlebot_radio_orbbec_ust10lx.urdf.xacro (robot description, xacro)
@@ -10,4 +10,6 @@
   <xacro:property name="CAMERA_H" value="0.197" />
   <xacro:property name="FOOT_H" value="0.02" />
+  <xacro:property name="min_angle" value="-2.09" />
+  <xacro:property name="max_angle" value="2.09" />
 <!--
 	- Distance from floot (base_footprint) to top_plate = 0.41 (41 cm)
@@ -30,5 +32,5 @@
       <origin xyz="-0.02 0.011 0.049" rpy="0 0 0" />
   </sensor_logitech_c920>
-  <sensor_hokuyo_ust10lx name="hokuyo" parent="base_link" >
+  <sensor_hokuyo_ust10lx name="hokuyo" parent="base_link" min_angle="${min_angle}" max_angle="${max_angle}">
 		<origin xyz="0.137 0 0.241" rpy="0 0 0" />
    </sensor_hokuyo_ust10lx>

File: turtlebot_description/robots/turtlebot_radio_xtion_ust10lx.urdf.xacro (robot description, xacro)
@@ -10,4 +10,6 @@
   <xacro:property name="CAMERA_H" value="0.197" />
   <xacro:property name="FOOT_H" value="0.02" />
+  <xacro:property name="min_angle" value="-2.09" />
+  <xacro:property name="max_angle" value="2.09" />
 <!--
 	- Distance from floot (base_footprint) to top_plate = 0.41 (41 cm)
@@ -30,5 +32,5 @@
       <origin xyz="-0.02 0.011 0.049" rpy="0 0 0" />
   </sensor_logitech_c920>
-  <sensor_hokuyo_ust10lx name="hokuyo" parent="base_link" >
+  <sensor_hokuyo_ust10lx name="hokuyo" parent="base_link" min_angle="${min_angle}" max_angle="${max_angle}">
 		<origin xyz="0.137 0 0.241" rpy="0 0 0" />
    </sensor_hokuyo_ust10lx>
