Commit message: turtlebot_description: adjusting model for intel r200 camera

File: turtlebot_description/robots/turtlebot_radio_r200_ust10lx.urdf.xacro (robot description, xacro)
@@ -24,9 +24,12 @@
   <stack_hexagons                 parent="base_link"/>
   <stack_bar				  	  parent="base_link"/>
-  <sensor_r200 name="radio" parent="telescopic_foot_link">
-      <origin xyz="0.02 0.0 ${2*FOOT_H-0.006}" rpy="0 0 0" />
+  <intel_r200_base prefix="radio_" parent="telescopic_foot_link">
+      <origin xyz="0.0 0.0 ${2*FOOT_H-0.006}" rpy="0 0 0" />
+  </intel_r200_base>
+  <sensor_r200 name="radio" parent="radio_r200_base_link">
+      <origin xyz="0.033 0.0 0.0313" rpy="0 0 0" />
   </sensor_r200>
-  <sensor_logitech_c920 prefix="rear" parent="telescopic_foot_link">
-      <origin xyz="-0.02 0.011 0.049" rpy="0 0 0" />
+  <sensor_logitech_c920 prefix="rear" parent="radio_r200_base_link">
+      <origin xyz="-0.07 0.0 0.0" rpy="0 0 0" />
   </sensor_logitech_c920>
   <sensor_hokuyo_ust10lx name="hokuyo" parent="base_link" >
@@ -34,5 +37,5 @@
    </sensor_hokuyo_ust10lx>
    <sensor_microphone_array name="radio" parent="plate_top_link" >
-		<origin xyz="0.1 0 0.006" rpy="0 0 0" />
+		<origin xyz="0.05 0 0.006" rpy="0 0 0" />
    </sensor_microphone_array>
    <!--screen name="radio" parent="plate_top_link" >

File: turtlebot_description/urdf/sensors/r200.urdf.xacro (robot description, xacro)
@@ -10,7 +10,7 @@
   <xacro:property name="r200_cam_offset_py" value="0.024" />
   <xacro:property name="r200_cam_offset_pz" value="0.005" />
-  <xacro:property name="r200_cam_rgb_px" value="0.005"/>
-  <xacro:property name="r200_cam_rgb_py" value="-0.018"/>
-  <xacro:property name="r200_cam_rgb_pz" value="0.013"/>
+  <xacro:property name="r200_cam_rgb_px" value="0.0"/>
+  <xacro:property name="r200_cam_rgb_py" value="-0.047"/>
+  <xacro:property name="r200_cam_rgb_pz" value="0.003"/>
   <xacro:property name="r200_cam_depth_offset" value="0.01"/>
   <xacro:macro name="sensor_r200" params="name parent *origin">
@@ -24,7 +24,8 @@
     <link name="${name}_cam_link">
       <visual>
-       <origin xyz="0 0 0" rpy="${M_PI/2} 0 ${M_PI/2}"/>
+       <!--origin xyz="0 0 0" rpy="${M_PI/2} 0 ${M_PI/2}"/-->
+       <origin xyz="0 0 0" rpy="0 0 0"/>
         <geometry>
-         <mesh filename="package://turtlebot_description/meshes/sensors/r200.dae" />
+         <mesh filename="package://turtlebot_description/meshes/sensors/intel_r200.dae" />
         </geometry>
       </visual>
@@ -32,10 +33,10 @@
         <origin xyz="0.0 0.0 0.0" rpy="0 0 0"/>
         <geometry>
-          <box size="0.130 0.567 0.118"/>
+          <mesh filename="package://turtlebot_description/meshes/sensors/intel_r200.dae" />
         </geometry>
       </collision>-->
       <!-- This inertial field needs doesn't contain reliable data!! -->
      <inertial>
-        <mass value="0.564" />
+        <mass value="0.100" />
         <origin xyz="0 0 0" />
         <inertia ixx="0.003881243" ixy="0.0" ixz="0.0"

File: turtlebot_description/urdf/turtlebot_library.urdf.xacro (robot description, xacro)
@@ -26,3 +26,4 @@
   <xacro:include filename="$(find turtlebot_description)/urdf/others/screen.urdf.xacro"/>
   <xacro:include filename="$(find turtlebot_description)/urdf/sensors/logitech_c920.urdf.xacro"/>
+  <xacro:include filename="$(find turtlebot_description)/urdf/others/intel_r200_base.urdf.xacro"/>
 </robot>
