Commit message: Added hokuyo ust10lx selectable with enviroment variable TURTLEBOT_LIDAR=urg04lx | ust10lx

File: turtlebot_description/robots/turtlebot_radio_orbbec_urg04.urdf.xacro (robot description, xacro)
@@ -5,5 +5,5 @@
     - Telescopic: telescopic
     - 3d Sensor : orbbec
-    - Laser		: hokuyo
+    - Laser		: urg04lx
 -->
 <robot name="turtlebot" xmlns:xacro="http://ros.org/wiki/xacro">

File: turtlebot_description/robots/turtlebot_radio_xtion_urg04.urdf.xacro (robot description, xacro)
@@ -5,5 +5,5 @@
     - Telescopic: telescopic
     - 3d Sensor : xtion
-    - Laser		: hokuyo
+    - Laser		: urg04lx
 -->
 <robot name="turtlebot" xmlns:xacro="http://ros.org/wiki/xacro">
@@ -27,4 +27,7 @@
 	<origin xyz="0.018 0.021 ${2*FOOT_H-0.006}" rpy="0 0 0" />
   </sensor_asus_xtion_pro_live>
+  <sensor_logitech_c920 prefix="rear" parent="telescopic_foot_link">
+      <origin xyz="-0.02 0.011 0.049" rpy="0 0 0" />
+  </sensor_logitech_c920>
   <sensor_hokuyo_urg04lx name="hokuyo" parent="base_link" >
 		<origin xyz="0.137 0 0.241" rpy="0 0 0" />

File: turtlebot_description/urdf/turtlebot_library.urdf.xacro (robot description, xacro)
@@ -19,4 +19,5 @@
   <xacro:include filename="$(find turtlebot_description)/urdf/sensors/asus_xtion_pro_live.urdf.xacro"/>
   <xacro:include filename="$(find turtlebot_description)/urdf/sensors/hokuyo_urg04lx.urdf.xacro" />
+  <xacro:include filename="$(find turtlebot_description)/urdf/sensors/hokuyo_ust10lx.urdf.xacro" />
   <xacro:include filename="$(find turtlebot_description)/urdf/sensors/orbbec_astra.urdf.xacro"/>
   <!-- Telescopic Bar -->

Commit message: description: setting the height of the camera to the new default position

File: turtlebot_description/robots/turtlebot_radio_orbbec_urg04.urdf.xacro (robot description, xacro)
@@ -8,5 +8,5 @@
 -->
 <robot name="turtlebot" xmlns:xacro="http://ros.org/wiki/xacro">
-  <xacro:property name="CAMERA_H" value="0.197" />
+  <xacro:property name="CAMERA_H" value="0.457" />
   <xacro:property name="FOOT_H" value="0.02" />
 <!--

File: turtlebot_description/robots/turtlebot_radio_orbbec_ust10lx.urdf.xacro (robot description, xacro)
@@ -8,5 +8,5 @@
 -->
 <robot name="turtlebot" xmlns:xacro="http://ros.org/wiki/xacro">
-  <xacro:property name="CAMERA_H" value="0.197" />
+  <xacro:property name="CAMERA_H" value="0.457" />
   <xacro:property name="FOOT_H" value="0.02" />
   <xacro:property name="min_angle" value="-2.09" />

File: turtlebot_description/robots/turtlebot_radio_xtion_urg04.urdf.xacro (robot description, xacro)
@@ -8,5 +8,5 @@
 -->
 <robot name="turtlebot" xmlns:xacro="http://ros.org/wiki/xacro">
-  <xacro:property name="CAMERA_H" value="0.197" />
+  <xacro:property name="CAMERA_H" value="0.457" />
   <xacro:property name="FOOT_H" value="0.02" />
 <!--

File: turtlebot_description/robots/turtlebot_radio_xtion_ust10lx.urdf.xacro (robot description, xacro)
@@ -8,5 +8,5 @@
 -->
 <robot name="turtlebot" xmlns:xacro="http://ros.org/wiki/xacro">
-  <xacro:property name="CAMERA_H" value="0.197" />
+  <xacro:property name="CAMERA_H" value="0.457" />
   <xacro:property name="FOOT_H" value="0.02" />
   <xacro:property name="min_angle" value="-2.09" />
