Commit message: Removed kinect frames

File: turtlebot_description/urdf/stacks/hexagons.urdf.xacro (robot description, xacro)
@@ -93,5 +93,5 @@
     </link>
   </xacro:macro>
-  <xacro:macro name="stack_3d_sensor_pole" params="parent number x_loc y_loc z_loc">
+  <!--xacro:macro name="stack_3d_sensor_pole" params="parent number x_loc y_loc z_loc">
     <joint name="pole_kinect_${number}_joint" type="fixed">
       <origin xyz="${x_loc} ${y_loc} ${z_loc}" rpy="0 0 0"/>
@@ -120,5 +120,5 @@
       </inertial>
     </link>
-  </xacro:macro>
+  </xacro:macro!-->
   <!--
     Stack macro - all the components relative transforms are made with respect
